File: signalgen/ddscore.sch (KiCad schematic (older format))
At the start: 10 parts, among them U8 AD9834

Commit message: First layout of DDS signal generator.
Changed lines of the file:
@@
 Connection ~ 5950 2400
 $Comp
-L GND #PWR53
+L GND #PWR057
 U 1 1 55389DF9
 P 5950 2700
-F 0 "#PWR53" H 5950 2450 50  0001 C CNN
+F 0 "#PWR057" H 5950 2450 50  0001 C CNN
 F 1 "GND" H 5950 2550 50  0000 C CNN
 F 2 "" H 5950 2700 60  0000 C CNN
@@
 $EndComp
 $Comp
-L GND #PWR55
+L GND #PWR058
 U 1 1 55389E11
 P 6200 2700
-F 0 "#PWR55" H 6200 2450 50  0001 C CNN
+F 0 "#PWR058" H 6200 2450 50  0001 C CNN
 F 1 "GND" H 6200 2550 50  0000 C CNN
 F 2 "" H 6200 2700 60  0000 C CNN
@@
 $EndComp
 $Comp
-L +5V #PWR57
+L +5V #PWR059
 U 1 1 55389E21
 P 6400 2400
-F 0 "#PWR57" H 6400 2250 50  0001 C CNN
+F 0 "#PWR059" H 6400 2250 50  0001 C CNN
 F 1 "+5V" H 6400 2540 50  0000 C CNN
 F 2 "" H 6400 2400 60  0000 C CNN
@@
 $EndComp
 $Comp
-L GND #PWR52
+L GND #PWR060
 U 1 1 55389EB1
 P 5950 2200
-F 0 "#PWR52" H 5950 1950 50  0001 C CNN
+F 0 "#PWR060" H 5950 1950 50  0001 C CNN
 F 1 "GND" H 5950 2050 50  0000 C CNN
 F 2 "" H 5950 2200 60  0000 C CNN
@@
 $EndComp
 $Comp
-L GND #PWR54
+L GND #PWR061
 U 1 1 55389EC6
 P 6200 2200
-F 0 "#PWR54" H 6200 1950 50  0001 C CNN
+F 0 "#PWR061" H 6200 1950 50  0001 C CNN
 F 1 "GND" H 6200 2050 50  0000 C CNN
 F 2 "" H 6200 2200 60  0000 C CNN
@@
 Connection ~ 5950 1900
 $Comp
-L +3.3V #PWR56
+L +3.3V #PWR062
 U 1 1 55389F87
 P 6400 1900
-F 0 "#PWR56" H 6400 1750 50  0001 C CNN
+F 0 "#PWR062" H 6400 1750 50  0001 C CNN
 F 1 "+3.3V" H 6400 2040 50  0000 C CNN
 F 2 "" H 6400 1900 60  0000 C CNN
@@
 $EndComp
 $Comp
-L GND #PWR49
+L GND #PWR063
 U 1 1 5538A0C3
 P 5100 2700
-F 0 "#PWR49" H 5100 2450 50  0001 C CNN
+F 0 "#PWR063" H 5100 2450 50  0001 C CNN
 F 1 "GND" H 5100 2550 50  0000 C CNN
 F 2 "" H 5100 2700 60  0000 C CNN
@@
 	6350 3150 6600 3150
 $Comp
-L +5V #PWR58
+L +5V #PWR064
 U 1 1 5538A2EF
 P 6600 2850
-F 0 "#PWR58" H 6600 2700 50  0001 C CNN
+F 0 "#PWR064" H 6600 2700 50  0001 C CNN
 F 1 "+5V" H 6600 2990 50  0000 C CNN
 F 2 "" H 6600 2850 60  0000 C CNN
@@
 $EndComp
 $Comp
-L GND #PWR60
+L GND #PWR065
 U 1 1 5538A41B
 P 6950 3550
-F 0 "#PWR60" H 6950 3300 50  0001 C CNN
+F 0 "#PWR065" H 6950 3300 50  0001 C CNN
 F 1 "GND" H 6950 3400 50  0000 C CNN
 F 2 "" H 6950 3550 60  0000 C CNN
@@
 	6400 3350 6350 3350
 $Comp
-L GND #PWR50
+L GND #PWR066
 U 1 1 5538A5FE
 P 5350 4450
-F 0 "#PWR50" H 5350 4200 50  0001 C CNN
+F 0 "#PWR066" H 5350 4200 50  0001 C CNN
 F 1 "GND" H 5350 4300 50  0000 C CNN
 F 2 "" H 5350 4450 60  0000 C CNN
@@
 $EndComp
 $Comp
-L GND #PWR51
+L GND #PWR067
 U 1 1 5538A620
 P 5750 4450
-F 0 "#PWR51" H 5750 4200 50  0001 C CNN
+F 0 "#PWR067" H 5750 4200 50  0001 C CNN
 F 1 "GND" H 5750 4300 50  0000 C CNN
 F 2 "" H 5750 4450 60  0000 C CNN
@@
 	4100 3650 4100 3850
 $Comp
-L GND #PWR48
+L GND #PWR068
 U 1 1 5538A87D
 P 4100 4150
-F 0 "#PWR48" H 4100 3900 50  0001 C CNN
+F 0 "#PWR068" H 4100 3900 50  0001 C CNN
 F 1 "GND" H 4100 4000 50  0000 C CNN
 F 2 "" H 4100 4150 60  0000 C CNN
@@
 $EndComp
 Wire Wire Line
-	6400 3550 6750 3550
-$Comp
-L GND #PWR59
+	6350 3550 6750 3550
+$Comp
+L GND #PWR069
 U 1 1 5538AD6F
 P 6750 3850
-F 0 "#PWR59" H 6750 3600 50  0001 C CNN
+F 0 "#PWR069" H 6750 3600 50  0001 C CNN
 F 1 "GND" H 6750 3700 50  0000 C CNN
 F 2 "" H 6750 3850 60  0000 C CNN
